Commit message: Update URDF to use it in RViz, switch visualization to RViz
For now, the frame is fixed on the first segment of the snake. This means, that only relative movement of the rest of the segments can be observed.

File: onshape_to_robot/snake/robot.urdf (robot description, URDF)
Before this commit: robot snake, 21 links, 20 joints
Links:
- link inner_adhesive_pad: geometry collision mesh filename=package://snake_sim/sdf/assets/inner_adhesive_pad.stl; visual mesh filename=package://snake_sim/sdf/assets/inner_adhesive_pad.stl
- link inner_adhesive_pad_2: geometry collision mesh filename=package://snake_sim/sdf/assets/inner_adhesive_pad.stl; visual mesh filename=package://snake_sim/sdf/assets/inner_adhesive_pad.stl
- link inner_adhesive_pad_3: geometry collision mesh filename=package://snake_sim/sdf/assets/inner_adhesive_pad.stl; visual mesh filename=package://snake_sim/sdf/assets/inner_adhesive_pad.stl
- link inner_adhesive_pad_4: geometry collision mesh filename=package://snake_sim/sdf/assets/inner_adhesive_pad.stl; visual mesh filename=package://snake_sim/sdf/assets/inner_adhesive_pad.stl
- link inner_adhesive_pad_5: geometry collision mesh filename=package://snake_sim/sdf/assets/inner_adhesive_pad.stl; visual mesh filename=package://snake_sim/sdf/assets/inner_adhesive_pad.stl
- link inner_adhesive_pad_6: geometry collision mesh filename=package://snake_sim/sdf/assets/inner_adhesive_pad.stl; visual mesh filename=package://snake_sim/sdf/assets/inner_adhesive_pad.stl
- link inner_adhesive_pad_7: geometry collision mesh filename=package://snake_sim/sdf/assets/inner_adhesive_pad.stl; visual mesh filename=package://snake_sim/sdf/assets/inner_adhesive_pad.stl
- link motor_with_no_arms: geometry collision mesh filename=package://snake_sim/sdf/assets/hn05_i101.stl; collision mesh filename=package://snake_sim/sdf/assets/mf128zz.stl
- link motor_with_onshape_mounting: geometry collision mesh filename=package://snake_sim/sdf/assets/hn05_i101.stl; collision mesh filename=package://snake_sim/sdf/assets/mf128zz.stl
- link motor_with_onshape_mounting_2: geometry collision mesh filename=package://snake_sim/sdf/assets/hn05_i101.stl; collision mesh filename=package://snake_sim/sdf/assets/mf128zz.stl
- link motor_with_onshape_mounting_3: geometry collision mesh filename=package://snake_sim/sdf/assets/hn05_i101.stl; collision mesh filename=package://snake_sim/sdf/assets/mf128zz.stl
- link motor_with_onshape_mounting_4: geometry collision mesh filename=package://snake_sim/sdf/assets/hn05_i101.stl; collision mesh filename=package://snake_sim/sdf/assets/mf128zz.stl
- link motor_with_onshape_mounting_5: geometry collision mesh filename=package://snake_sim/sdf/assets/hn05_i101.stl; collision mesh filename=package://snake_sim/sdf/assets/mf128zz.stl
- link motor_with_onshape_mounting_6: geometry collision mesh filename=package://snake_sim/sdf/assets/hn05_i101.stl; collision mesh filename=package://snake_sim/sdf/assets/mf128zz.stl
- link outer_adhesive_pad: geometry collision mesh filename=package://snake_sim/sdf/assets/outer_adhesive_pad.stl; visual mesh filename=package://snake_sim/sdf/assets/outer_adhesive_pad.stl
- link outer_adhesive_pad_2: geometry collision mesh filename=package://snake_sim/sdf/assets/outer_adhesive_pad.stl; visual mesh filename=package://snake_sim/sdf/assets/outer_adhesive_pad.stl
- link outer_adhesive_pad_3: geometry collision mesh filename=package://snake_sim/sdf/assets/outer_adhesive_pad.stl; visual mesh filename=package://snake_sim/sdf/assets/outer_adhesive_pad.stl
- link outer_adhesive_pad_4: geometry collision mesh filename=package://snake_sim/sdf/assets/outer_adhesive_pad.stl; visual mesh filename=package://snake_sim/sdf/assets/outer_adhesive_pad.stl
- link outer_adhesive_pad_5: geometry collision mesh filename=package://snake_sim/sdf/assets/outer_adhesive_pad.stl; visual mesh filename=package://snake_sim/sdf/assets/outer_adhesive_pad.stl
- link outer_adhesive_pad_6: geometry collision mesh filename=package://snake_sim/sdf/assets/outer_adhesive_pad.stl; visual mesh filename=package://snake_sim/sdf/assets/outer_adhesive_pad.stl
- link outer_adhesive_pad_7: geometry collision mesh filename=package://snake_sim/sdf/assets/outer_adhesive_pad.stl; visual mesh filename=package://snake_sim/sdf/assets/outer_adhesive_pad.stl

File: urdf/snake.urdf (robot description, URDF)
Before this commit: robot snake, 21 links, 20 joints
Links:
- link inner_adhesive_pad: geometry collision mesh filename=package://snake_sim/sdf/assets/inner_adhesive_pad.stl; visual mesh filename=package://snake_sim/sdf/assets/inner_adhesive_pad.stl
- link inner_adhesive_pad_2: geometry collision mesh filename=package://snake_sim/sdf/assets/inner_adhesive_pad.stl; visual mesh filename=package://snake_sim/sdf/assets/inner_adhesive_pad.stl
- link inner_adhesive_pad_3: geometry collision mesh filename=package://snake_sim/sdf/assets/inner_adhesive_pad.stl; visual mesh filename=package://snake_sim/sdf/assets/inner_adhesive_pad.stl
- link inner_adhesive_pad_4: geometry collision mesh filename=package://snake_sim/sdf/assets/inner_adhesive_pad.stl; visual mesh filename=package://snake_sim/sdf/assets/inner_adhesive_pad.stl
- link inner_adhesive_pad_5: geometry collision mesh filename=package://snake_sim/sdf/assets/inner_adhesive_pad.stl; visual mesh filename=package://snake_sim/sdf/assets/inner_adhesive_pad.stl
- link inner_adhesive_pad_6: geometry collision mesh filename=package://snake_sim/sdf/assets/inner_adhesive_pad.stl; visual mesh filename=package://snake_sim/sdf/assets/inner_adhesive_pad.stl
- link inner_adhesive_pad_7: geometry collision mesh filename=package://snake_sim/sdf/assets/inner_adhesive_pad.stl; visual mesh filename=package://snake_sim/sdf/assets/inner_adhesive_pad.stl
- link motor_with_no_arms: geometry collision mesh filename=package://snake_sim/sdf/assets/hn05_i101.stl; collision mesh filename=package://snake_sim/sdf/assets/mf128zz.stl
- link motor_with_onshape_mounting: geometry collision mesh filename=package://snake_sim/sdf/assets/hn05_i101.stl; collision mesh filename=package://snake_sim/sdf/assets/mf128zz.stl
- link motor_with_onshape_mounting_2: geometry collision mesh filename=package://snake_sim/sdf/assets/hn05_i101.stl; collision mesh filename=package://snake_sim/sdf/assets/mf128zz.stl
- link motor_with_onshape_mounting_3: geometry collision mesh filename=package://snake_sim/sdf/assets/hn05_i101.stl; collision mesh filename=package://snake_sim/sdf/assets/mf128zz.stl
- link motor_with_onshape_mounting_4: geometry collision mesh filename=package://snake_sim/sdf/assets/hn05_i101.stl; collision mesh filename=package://snake_sim/sdf/assets/mf128zz.stl
- link motor_with_onshape_mounting_5: geometry collision mesh filename=package://snake_sim/sdf/assets/hn05_i101.stl; collision mesh filename=package://snake_sim/sdf/assets/mf128zz.stl
- link motor_with_onshape_mounting_6: geometry collision mesh filename=package://snake_sim/sdf/assets/hn05_i101.stl; collision mesh filename=package://snake_sim/sdf/assets/mf128zz.stl
- link outer_adhesive_pad: geometry collision mesh filename=package://snake_sim/sdf/assets/outer_adhesive_pad.stl; visual mesh filename=package://snake_sim/sdf/assets/outer_adhesive_pad.stl
- link outer_adhesive_pad_2: geometry collision mesh filename=package://snake_sim/sdf/assets/outer_adhesive_pad.stl; visual mesh filename=package://snake_sim/sdf/assets/outer_adhesive_pad.stl
- link outer_adhesive_pad_3: geometry collision mesh filename=package://snake_sim/sdf/assets/outer_adhesive_pad.stl; visual mesh filename=package://snake_sim/sdf/assets/outer_adhesive_pad.stl
- link outer_adhesive_pad_4: geometry collision mesh filename=package://snake_sim/sdf/assets/outer_adhesive_pad.stl; visual mesh filename=package://snake_sim/sdf/assets/outer_adhesive_pad.stl
- link outer_adhesive_pad_5: geometry collision mesh filename=package://snake_sim/sdf/assets/outer_adhesive_pad.stl; visual mesh filename=package://snake_sim/sdf/assets/outer_adhesive_pad.stl
- link outer_adhesive_pad_6: geometry collision mesh filename=package://snake_sim/sdf/assets/outer_adhesive_pad.stl; visual mesh filename=package://snake_sim/sdf/assets/outer_adhesive_pad.stl
- link outer_adhesive_pad_7: geometry collision mesh filename=package://snake_sim/sdf/assets/outer_adhesive_pad.stl; visual mesh filename=package://snake_sim/sdf/assets/outer_adhesive_pad.stl
